File: DaNumPad Glow/matrix.sch (KiCad schematic (older format))
At the start: 56 parts, among them SW1 SW_Push, SW10 SW_Push, SW11 SW_Push, SW12 SW_Push, SW13 SW_Push, SW14 SW_Push, SW15 SW_Push, SW16 SW_Push, SW17 SW_Push, SW18 SW_Push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

Commit message: Glow version redesign
For now, it's 17 keys only.
Connections:
- net Col_0: now also ENC1.S2; no longer ENC1.S1
- net Enc_0: now also ENC1.S1; no longer ENC1.S2
Changed lines of the file:
@@
 $Descr A4 11693 8268
 encoding utf-8
-Sheet 2 2
+Sheet 2 3
 Title ""
 Date ""
@@
 	0    1    1    0
 $EndComp
-Text GLabel 7050 1700 2    50   Input ~ 0
+Text GLabel 7050 1500 2    50   Input ~ 0
 Enc_0
 Text GLabel 7050 2700 2    50   Input ~ 0
@@
 Wire Wire Line
 	7050 1700 6950 1700
-Text GLabel 7050 1500 2    50   Input ~ 0
+Text GLabel 7050 1700 2    50   Input ~ 0
 Col_0
 Wire Wire Line
