File: DaNumPad Glow/DaNumPad Glow 17.kicad_pcb (KiCad board)
At the start: 2 copper layers, 100 x 95.3 mm, 102 parts, among them J1 USB_C_Receptacle_USB2.0, J4 Conn_01x06, SW1 SW_Push, SW10 SW_Push, SW11 SW_Push, SW13 SW_Push, SW14 SW_Push, SW15 SW_Push, SW19 SW_Push, SW2 SW_Push, SW21 SW_Push, SW22 SW_Push, SW23 SW_Push, SW24 TS-A002, SW3 SW_Push, SW4 SW_Push, SW5 SW_Push, SW6 SW_Push, SW7 SW_Push, SW9 SW_Push, U1 SRV05-4, U5 ATmega32U4, X2 X322516MLB4SI

Commit message: Finalized licensing on PCB files
Routing:
- net Row_2: track 87.1 -> 82.3 mm
Other:
- board text added: "DaNumPad - Glow v1.00 Markus Knutsson 2021 https://github.com/TweetyDaBird Licensed under CERN-OHL-S v2+ JLCJLCJLCJLC"

Commit message: Cleanup of silkscreen
Parts:
- C4: renamed from C16; value 0.1uF -> 100nF
- C5: renamed from C17; value 0.1uF -> 100nF
- C6: renamed from C18; value 0.1uF -> 100nF
- C7: renamed from C19; value 0.1uF -> 100nF
- C8: renamed from C20; value 0.1uF -> 100nF
- U2: renamed from U5; footprint Package_DFN_QFN:QFN-44-1EP_7x7mm_P0.5mm_EP5.15x5.15mm -> Package_DFN_QFN:QFN-44-1EP_7x7mm_P0.5mm_EP5.15x5.15mm_ThermalVias
- renumbered C13 to C1, C1 to C10, C2 to C11, C11 to C12, C12 to C13, C22 to C14, C3 to C15, C4 to C16, C5 to C17, C6 to C18, C23 to C19, C14 to C2, C24 to C20, C25 to C21, C26 to C22, C7 to C23, C8 to C24, C9 to C25, C10 to C26, C15 to C3, C21 to C9, D13 to D12, D14 to D13, D15 to D14, D17 to D15, D19 to D16, D20 to D17, D12 to D8, J4 to J2, LED_3 to LED_1, LED_4 to LED_2, R8 to R3, R10 to R4, R11 to R5, R12 to R6, R13 to R7, RGB13 to RGB12, RGB14 to RGB13, RGB15 to RGB14, RGB16 to RGB15, RGB17 to RGB16, RGB18 to RGB17, SW24 to SW1, SW9 to SW10, SW10 to SW11, SW11 to SW12, SW23 to SW16, SW19 to SW17, SW22 to SW18, SW1 to SW2, SW2 to SW3, SW3 to SW4, SW4 to SW5, SW5 to SW6, SW6 to SW7, SW7 to SW8, SW21 to SW9, X2 to X1
Connections:
- RGB1 pad 3: (no net) -> RGB
- U2 pad 1: (no net) -> RGB
Routing:
- net RGB: track 0.00 -> 22.3 mm, vias 0 -> 1
- net VCC: track 538.9 -> 539.8 mm
