File: DaNumPad Glow/matrix 17.sch (KiCad schematic (older format))
At the start: 75 parts, among them SW1 SW_Push, SW10 SW_Push, SW11 SW_Push, SW13 SW_Push, SW14 SW_Push, SW15 SW_Push, SW19 SW_Push, SW2 SW_Push, SW21 SW_Push, SW22 SW_Push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

Commit message: Cleanup of silkscreen
Parts:
- C10: renamed from C1; JLPCB Type (none) -> Basic; LCSC (none) -> C14663; Manufacturer_Name (none) -> YAGEO; Manufacturer_Part_Number (none) -> CC0603KRX7R9BB104; fit_field (none) -> DNF
- C11: renamed from C2; JLPCB Type (none) -> Basic; LCSC (none) -> C14663; Manufacturer_Name (none) -> YAGEO; Manufacturer_Part_Number (none) -> CC0603KRX7R9BB104; fit_field (none) -> DNF
- C12: renamed from C11; JLPCB Type (none) -> Basic; LCSC (none) -> C14663; Manufacturer_Name (none) -> YAGEO; Manufacturer_Part_Number (none) -> CC0603KRX7R9BB104; fit_field (none) -> DNF
- C13: renamed from C12; JLPCB Type (none) -> Basic; LCSC (none) -> C14663; Manufacturer_Name (none) -> YAGEO; Manufacturer_Part_Number (none) -> CC0603KRX7R9BB104; fit_field (none) -> DNF
- C14: renamed from C22; JLPCB Type (none) -> Basic; LCSC (none) -> C14663; Manufacturer_Name (none) -> YAGEO; Manufacturer_Part_Number (none) -> CC0603KRX7R9BB104; fit_field (none) -> DNF
- C15: renamed from C3; JLPCB Type (none) -> Basic; LCSC (none) -> C14663; Manufacturer_Name (none) -> YAGEO; Manufacturer_Part_Number (none) -> CC0603KRX7R9BB104; fit_field (none) -> DNF
- C16: renamed from C4; JLPCB Type (none) -> Basic; LCSC (none) -> C14663; Manufacturer_Name (none) -> YAGEO; Manufacturer_Part_Number (none) -> CC0603KRX7R9BB104; fit_field (none) -> DNF
- C17: renamed from C5; JLPCB Type (none) -> Basic; LCSC (none) -> C14663; Manufacturer_Name (none) -> YAGEO; Manufacturer_Part_Number (none) -> CC0603KRX7R9BB104; fit_field (none) -> DNF
- C18: renamed from C6; JLPCB Type (none) -> Basic; LCSC (none) -> C14663; Manufacturer_Name (none) -> YAGEO; Manufacturer_Part_Number (none) -> CC0603KRX7R9BB104; fit_field (none) -> DNF
- C19: renamed from C23; JLPCB Type (none) -> Basic; LCSC (none) -> C14663; Manufacturer_Name (none) -> YAGEO; Manufacturer_Part_Number (none) -> CC0603KRX7R9BB104; fit_field (none) -> DNF
- C20: renamed from C24; JLPCB Type (none) -> Basic; LCSC (none) -> C14663; Manufacturer_Name (none) -> YAGEO; Manufacturer_Part_Number (none) -> CC0603KRX7R9BB104; fit_field (none) -> DNF
- C21: renamed from C25; JLPCB Type (none) -> Basic; LCSC (none) -> C14663; Manufacturer_Name (none) -> YAGEO; Manufacturer_Part_Number (none) -> CC0603KRX7R9BB104; fit_field (none) -> DNF
- C22: renamed from C26; JLPCB Type (none) -> Basic; LCSC (none) -> C14663; Manufacturer_Name (none) -> YAGEO; Manufacturer_Part_Number (none) -> CC0603KRX7R9BB104; fit_field (none) -> DNF
- C23: renamed from C7; JLPCB Type (none) -> Basic; LCSC (none) -> C14663; Manufacturer_Name (none) -> YAGEO; Manufacturer_Part_Number (none) -> CC0603KRX7R9BB104; fit_field (none) -> DNF
- C24: renamed from C8; JLPCB Type (none) -> Basic; LCSC (none) -> C14663; Manufacturer_Name (none) -> YAGEO; Manufacturer_Part_Number (none) -> CC0603KRX7R9BB104; fit_field (none) -> DNF
- C25: renamed from C9; JLPCB Type (none) -> Basic; LCSC (none) -> C14663; Manufacturer_Name (none) -> YAGEO; Manufacturer_Part_Number (none) -> CC0603KRX7R9BB104; fit_field (none) -> DNF
- C26: renamed from C10; JLPCB Type (none) -> Basic; LCSC (none) -> C14663; Manufacturer_Name (none) -> YAGEO; Manufacturer_Part_Number (none) -> CC0603KRX7R9BB104; fit_field (none) -> DNF
- D1, D10, D11, D2, D3, D4, D5, D6, D7, D9: JLPCB Type (none) -> Basic; fit_field (none) -> DNF
- D12: renamed from D13; JLPCB Type (none) -> Basic; fit_field (none) -> DNF
- D13: renamed from D14; JLPCB Type (none) -> Basic; fit_field (none) -> DNF
- D14: renamed from D15; JLPCB Type (none) -> Basic; fit_field (none) -> DNF
- D15: renamed from D17; JLPCB Type (none) -> Basic; fit_field (none) -> DNF
- D16: renamed from D19; JLPCB Type (none) -> Basic; fit_field (none) -> DNF
- D17: renamed from D20; JLPCB Type (none) -> Basic; fit_field (none) -> DNF
- D8: renamed from D12; JLPCB Type (none) -> Basic; fit_field (none) -> DNF
- H1, H2, H3, H4, RGB1, RGB10, RGB11, RGB2, RGB3, RGB4, RGB5, RGB6, RGB7, RGB8, RGB9, ST1, ST2, ST3, SW13, SW14, SW15: fit_field (none) -> DNF
- RGB12: renamed from RGB13; fit_field (none) -> DNF
- RGB13: renamed from RGB14; fit_field (none) -> DNF
- RGB14: renamed from RGB15; fit_field (none) -> DNF
- RGB15: renamed from RGB16; fit_field (none) -> DNF
- RGB16: renamed from RGB17; fit_field (none) -> DNF
- RGB17: renamed from RGB18; fit_field (none) -> DNF
- SW10: renamed from SW9; fit_field (none) -> DNF
- SW11: renamed from SW10; fit_field (none) -> DNF
- SW12: renamed from SW11; fit_field (none) -> DNF
- SW16: renamed from SW23; fit_field (none) -> DNF
- SW17: renamed from SW19; fit_field (none) -> DNF
- SW18: renamed from SW22; fit_field (none) -> DNF
- SW2: renamed from SW1; fit_field (none) -> DNF
- SW3: renamed from SW2; fit_field (none) -> DNF
- SW4: renamed from SW3; fit_field (none) -> DNF
- SW5: renamed from SW4; fit_field (none) -> DNF
- SW6: renamed from SW5; fit_field (none) -> DNF
- SW7: renamed from SW6; fit_field (none) -> DNF
- SW8: renamed from SW7; fit_field (none) -> DNF
- SW9: renamed from SW21; fit_field (none) -> DNF
Connections:
- net LED renamed RGB
