File: DaNumPad unWired/DaNumPad unWired.kicad_pcb (KiCad board)
At the start: 2 copper layers, 100 x 95.3 mm, 92 parts, among them J1 USB_C_Receptacle_USB2.0, J2 Conn_01x02, J3 Conn_01x04, Q1 SI2301CDS-T1-GE3, SW1 SW_Push, SW10 SW_Push, SW11 SW_Push, SW12 SW_Push, SW13 SW_Push, SW14 SW_Push, SW15 SW_Push, SW16 SW_Push, SW17 SW_Push, SW18 SW_Push, SW19 SW_Push, SW2 SW_Push, SW20 SW_Push, SW21 SW_Push, SW22 SW_Push, SW23 SW_Push, SW24 TS-A002, SW3 SW_Push, SW4 SW_Push, SW5 SW_Push, SW6 SW_Push, SW7 SW_Push, SW8 SW_Push, SW9 SW_Push, U1 SRV05-4, U2 nRF52840_holyiot_18010, U3 TP4056, U4 XC6206PxxxMR-Regulator_Linear

Commit message: Added silkscreen and PCB Plates
Parts:
- removed BT1: Battery_Cell, Keyboard Library:Lipo_battery_501528_1S_150mAh
Routing:
- net GND: vias 20 -> 21
Other:
- board text added: "DaNumPad unWired v1.00 Markus Knutsson 2021 https://github.com/TweetyDaBird Licensed under CERN-OHL-S v2+ JLCJLCJLCJLC"
