File: DaNumPad Glow 20/matrix.sch (KiCad schematic (older format))
At the start: 56 parts, among them SW1 SW_Push, SW10 SW_Push, SW11 SW_Push, SW12 SW_Push, SW13 SW_Push, SW14 SW_Push, SW15 SW_Push, SW16 SW_Push, SW17 SW_Push, SW18 SW_Push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

Commit message: Added Glow 20 key version
Parts:
- removed ST1, ST2, ST3: Stabilizer_2u_MX, keyswitches:Stabilizer_MX_2u, symbol Keyboard_Library:Stabilizer_2u_MX
- removed SW21, SW22, SW23: SW_Push, keyswitches:Kailh_socket_MX_RGB, symbol Switch:SW_Push
- renumbered C9 to C27, C10 to C28, C11 to C29, C12 to C30
Connections:
- net Alt_Enter: no longer names the net of D20.2 (A), SW20.2
- net Alt_Plus: no longer names the net of D12.2 (A), SW12.2
Changed lines of the file:
@@
 encoding utf-8
 Sheet 2 3
-Title ""
-Date ""
-Rev ""
-Comp ""
-Comment1 ""
-Comment2 ""
+Title "DaNumPad - Glow 20"
+Date "2021-09-09"
+Rev "v1.0"
+Comp "Markus Knutsson <markus.knutsson@tweety.se>"
+Comment1 "https://github.com/TweetyDaBird"
+Comment2 "Licensed under CERN-OHL-S v2 or superseding version"
 Comment3 ""
 Comment4 ""
@@
 Text GLabel 1950 4950 0    50   Input ~ 0
 Row_4
-$Comp
-L Switch:SW_Push SW21
-U 1 1 615FD54C
-P 3150 5650
-F 0 "SW21" H 3150 5935 50  0000 C CNN
-F 1 "SW_Push" H 3150 5844 50  0000 C CNN
-F 2 "keyswitches:Kailh_socket_MX_RGB" H 3150 5850 50  0001 C CNN
-F 3 "~" H 3150 5850 50  0001 C CNN
-	1    3150 5650
-	-1   0    0    -1
-$EndComp
 Wire Wire Line
 	3950 3550 4550 3550
-$Comp
-L Switch:SW_Push SW22
-U 1 1 61603E38
-P 3150 6150
-F 0 "SW22" H 3150 6435 50  0000 C CNN
-F 1 "SW_Push" H 3150 6344 50  0000 C CNN
-F 2 "keyswitches:Kailh_socket_MX_RGB" H 3150 6350 50  0001 C CNN
-F 3 "~" H 3150 6350 50  0001 C CNN
-	1    3150 6150
-	-1   0    0    -1
-$EndComp
-$Comp
-L Switch:SW_Push SW23
-U 1 1 61607A79
-P 3150 6650
-F 0 "SW23" H 3150 6935 50  0000 C CNN
-F 1 "SW_Push" H 3150 6844 50  0000 C CNN
-F 2 "keyswitches:Kailh_socket_MX_RGB" H 3150 6850 50  0001 C CNN
-F 3 "~" H 3150 6850 50  0001 C CNN
-	1    3150 6650
-	1    0    0    -1
-$EndComp
 Wire Wire Line
 	4100 3250 4100 3950
-Text GLabel 2950 5650 0    50   Input ~ 0
-Col_3
-Text GLabel 2950 6150 0    50   Input ~ 0
-Col_3
-Text GLabel 2950 6650 0    50   Input ~ 0
-Col_0
-Text GLabel 3350 6650 2    50   Input ~ 0
-Alt_0
 Text GLabel 2800 4600 1    50   Input ~ 0
 Alt_0
@@
 	2800 4650 2750 4650
 Connection ~ 2750 4650
-Text GLabel 4650 4650 1    50   Input ~ 0
-Alt_Enter
-Wire Wire Line
-	4650 4650 4550 4650
-Connection ~ 4550 4650
-Text GLabel 3350 6150 2    50   Input ~ 0
-Alt_Enter
-Text GLabel 3350 5650 2    50   Input ~ 0
-Alt_Plus
-Text GLabel 4650 3250 1    50   Input ~ 0
-Alt_Plus
-Wire Wire Line
-	4650 3250 4550 3250
-Connection ~ 4550 3250
 Text GLabel 2800 1800 1    50   Input ~ 0
 Enc_0
@@
 $EndComp
 $Comp
-L power:GND #PWR017
+L power:GND #PWR047
 U 1 1 6167A73B
 P 6650 1900
-F 0 "#PWR017" H 6650 1650 50  0001 C CNN
+F 0 "#PWR047" H 6650 1650 50  0001 C CNN
 F 1 "GND" H 6655 1727 50  0000 C CNN
 F 2 "" H 6650 1900 50  0001 C CNN
@@
 $EndComp
 $Comp
-L power:GND #PWR019
+L power:GND #PWR049
 U 1 1 6167EEF6
 P 6650 2900
-F 0 "#PWR019" H 6650 2650 50  0001 C CNN
+F 0 "#PWR049" H 6650 2650 50  0001 C CNN
 F 1 "GND" H 6655 2727 50  0000 C CNN
 F 2 "" H 6650 2900 50  0001 C CNN
@@
 Enc_1_B
 $Comp
-L Device:C_Small C9
+L Device:C_Small C27
 U 1 1 6168566A
 P 5900 1500
-F 0 "C9" H 5992 1546 50  0000 L CNN
+F 0 "C27" H 5992 1546 50  0000 L CNN
 F 1 "100nF" H 5992 1455 50  0000 L CNN
 F 2 "Capacitor_SMD:C_0603_1608Metric" H 5900 1500 50  0001 C CNN
@@
 $EndComp
 $Comp
-L Device:C_Small C10
+L Device:C_Small C28
 U 1 1 61691868
 P 5900 1700
-F 0 "C10" H 5992 1746 50  0000 L CNN
+F 0 "C28" H 5992 1746 50  0000 L CNN
 F 1 "100nF" H 5992 1655 50  0000 L CNN
 F 2 "Capacitor_SMD:C_0603_1608Metric" H 5900 1700 50  0001 C CNN
@@
 Connection ~ 5900 1800
 $Comp
-L power:GND #PWR016
+L power:GND #PWR046
 U 1 1 6169F665
 P 5750 1600
-F 0 "#PWR016" H 5750 1350 50  0001 C CNN
+F 0 "#PWR046" H 5750 1350 50  0001 C CNN
 F 1 "GND" V 5755 1472 50  0000 R CNN
 F 2 "" H 5750 1600 50  0001 C CNN
@@
 $EndComp
 $Comp
-L Device:C_Small C11
+L Device:C_Small C29
 U 1 1 616AA649
 P 5900 2500
-F 0 "C11" H 5992 2546 50  0000 L CNN
+F 0 "C29" H 5992 2546 50  0000 L CNN
 F 1 "100nF" H 5992 2455 50  0000 L CNN
 F 2 "Capacitor_SMD:C_0603_1608Metric" H 5900 2500 50  0001 C CNN
@@
 $EndComp
 $Comp
-L Device:C_Small C12
+L Device:C_Small C30
 U 1 1 616AA64F
 P 5900 2700
-F 0 "C12" H 5992 2746 50  0000 L CNN
+F 0 "C30" H 5992 2746 50  0000 L CNN
 F 1 "100nF" H 5992 2655 50  0000 L CNN
 F 2 "Capacitor_SMD:C_0603_1608Metric" H 5900 2700 50  0001 C CNN
@@
 Connection ~ 5900 2800
 $Comp
-L power:GND #PWR018
+L power:GND #PWR048
 U 1 1 616B0A68
 P 5750 2600
-F 0 "#PWR018" H 5750 2350 50  0001 C CNN
+F 0 "#PWR048" H 5750 2350 50  0001 C CNN
 F 1 "GND" V 5755 2472 50  0000 R CNN
 F 2 "" H 5750 2600 50  0001 C CNN
@@
 	1    0    0    -1
 $EndComp
-$Comp
-L Keyboard_Library:Stabilizer_2u_MX ST1
-U 1 1 616D425C
-P 8800 4950
-F 0 "ST1" H 8986 5003 60  0000 L CNN
-F 1 "Stabilizer_2u_MX" H 8986 4897 60  0000 L CNN
-F 2 "keyswitches:Stabilizer_MX_2u" H 8800 4950 60  0001 C CNN
-F 3 "" H 8800 4950 60  0001 C CNN
-	1    8800 4950
-	1    0    0    -1
-$EndComp
-$Comp
-L Keyboard_Library:Stabilizer_2u_MX ST2
-U 1 1 616D4C96
-P 8800 5350
-F 0 "ST2" H 8986 5403 60  0000 L CNN
-F 1 "Stabilizer_2u_MX" H 8986 5297 60  0000 L CNN
-F 2 "keyswitches:Stabilizer_MX_2u" H 8800 5350 60  0001 C CNN
-F 3 "" H 8800 5350 60  0001 C CNN
-	1    8800 5350
-	1    0    0    -1
-$EndComp
-$Comp
-L Keyboard_Library:Stabilizer_2u_MX ST3
-U 1 1 616D52C0
-P 8800 5800
-F 0 "ST3" H 8986 5853 60  0000 L CNN
-F 1 "Stabilizer_2u_MX" H 8986 5747 60  0000 L CNN
-F 2 "keyswitches:Stabilizer_MX_2u" H 8800 5800 60  0001 C CNN
-F 3 "" H 8800 5800 60  0001 C CNN
-	1    8800 5800
-	1    0    0    -1
-$EndComp
